Commit message: write linkage kinematics for inspire hand

File: inspire_tactile_hand/urdf/inspire_tactile_hand.urdf (robot description, URDF)
Before this commit: robot inspire_tactile_hand, 32 links, 31 joints
Links:
- removed link base_link
- added link hand_base_link, mass 0.091809; collision mesh filename=package://inspire_tactile_hand/meshes/base_link.STL; visual mesh filename=package://inspire_tactile_hand/meshes/base_link.STL
Joints:
- joint fixed: child base_link -> hand_base_link
- joint joint001: parent base_link -> hand_base_link
- joint joint005: parent base_link -> hand_base_link
- joint joint401: parent base_link -> hand_base_link
- joint joint601: parent base_link -> hand_base_link
- joint joint605: parent base_link -> hand_base_link
- joint joint701: parent base_link -> hand_base_link
- joint joint705: parent base_link -> hand_base_link
- joint joint801: parent base_link -> hand_base_link
- joint joint805: parent base_link -> hand_base_link
